Commit message: description: add Purple color for camera bounding box
Signed-off-by: Jean Laneurit <jean.laneurit@inrae.fr>

File: romea_camera_description/urdf/camera.xacro (robot description, xacro)
@@ -80,4 +80,5 @@
         </joint>
         <gazebo reference="${link_name}">
+          <material>Gazebo/Purple</material>
           <sensor type="camera" name="${prefix}${name}">
             <update_rate>${frame_rate}</update_rate>

Commit message: description: add camera_simulation.xacro in order to support ignition gazebo and isaac sim
Signed-off-by: Jean Laneurit <jean.laneurit@inrae.fr>

File: romea_camera_description/urdf/camera.xacro (robot description, xacro)
@@ -16,23 +16,25 @@
         <xacro:property name="optical_joint_name"
           value="${prefix}${name}_optical_joint"/>
-        <xacro:property name="image_width"
-          value="${configuration['image_width']}" />
-        <xacro:property name="image_height"
-          value="${configuration['image_height']}" />
-        <xacro:property name="horizontal_fov"
-          value="${configuration['horizontal_fov']}" />
-        <xacro:property name="frame_rate"
-          value="${configuration['frame_rate']}" />
-        <xacro:property name="mass" value="${geometry['mass']}" />
-        <xacro:property name="aabb" value="${geometry['aabb']}" />
-        <xacro:property name="aabb_length" value="${geometry['aabb']['length']}" />
-        <xacro:property name="aabb_width" value="${geometry['aabb']['width']}" />
-        <xacro:property name="aabb_height" value="${geometry['aabb']['height']}" />
-        <xacro:property name="aabb_center" value="${geometry['aabb']['center']}" />
+        <xacro:property name="mass"
+          value="${geometry['mass']}" />
+        <xacro:property name="aabb"
+          value="${geometry['aabb']}" />
+        <xacro:property name="aabb_length"
+          value="${geometry['aabb']['length']}" />
+        <xacro:property name="aabb_width"
+          value="${geometry['aabb']['width']}" />
+        <xacro:property name="aabb_height"
+          value="${geometry['aabb']['height']}" />
+        <xacro:property name="aabb_center"
+          value="${geometry['aabb']['center']}" />
         <xacro:if value="${mesh_visual == True and 'mesh' in geometry}">
-        <xacro:property name="mesh_xyz" value="${geometry['mesh']['xyz']}" />
-        <xacro:property name="mesh_rpy" value="${geometry['mesh']['rpy']}" />
-        <xacro:property name="mesh_scale" value="${geometry['mesh']['scale']}" />
-        <xacro:property name="mesh_filename" value="${geometry['mesh']['filename']}" />
+          <xacro:property name="mesh_xyz"
+            value="${geometry['mesh']['xyz']}" />
+          <xacro:property name="mesh_rpy"
+            value="${geometry['mesh']['rpy']}" />
+          <xacro:property name="mesh_scale"
+            value="${geometry['mesh']['scale']}" />
+          <xacro:property name="mesh_filename"
+            value="${geometry['mesh']['filename']}" />
         </xacro:if>
         <link name="${link_name}">
@@ -79,48 +81,7 @@
             <child link="${optical_frame_name}"/>
         </joint>
-        <gazebo reference="${link_name}">
-          <material>Gazebo/Purple</material>
-          <sensor type="camera" name="${prefix}${name}">
-            <update_rate>${frame_rate}</update_rate>
-            <camera>
-              <pose>0 0 0 0 0 0</pose>
-              <horizontal_fov>${horizontal_fov}</horizontal_fov>
-              <image>
-                <width>${image_width} </width>
-                <height>${image_height}</height>
-                <format>R8G8B8</format>
-              </image>
-              <clip>
-                <near>0.01</near>
-                <far>100</far>
-              </clip>
-              <!-- <noise>
-                <type>gaussian</type>
-                <mean>0.0</mean>
-                <stddev>0.007</stddev>
-              </noise>
-              <distortion>
-                <k1>0.0</k1>
-                <k2>0.0</k2>
-                <k3>0.0</k3>
-                <p1>0.0</p1>
-                <p2>0.0</p2>
-                <center>0.5 0.5</center>
-              </distortion> -->
-            </camera>
-            <plugin name="driver" filename="libgazebo_ros_camera.so">
-                <ros>
-                  <namespace>${ros_namespace}</namespace>
-                  <remapping>camera/image_raw:=image_raw</remapping>
-                  <remapping>camera/camera_info:=camera_info</remapping>
-                  <remapping>camera/image_raw/compressed:=image_raw/compressed</remapping>
-                  <remapping>camera/image_raw/compressedDepth:=image_raw/compressedDepth</remapping>
-                  <remapping>camera/image_raw/theora:=image_raw/theora</remapping>
-                </ros>
-                <camera_name>camera</camera_name>
-                <hack_baseline>0.07</hack_baseline>
-            </plugin>
-          </sensor>
-        </gazebo>
+        <xacro:if value="${'simulation' in mode}">
+          <xacro:include filename="$(find romea_camera_description)/urdf/camera.simulation.xacro" />
+        </xacro:if>
     </xacro:macro>
 </robot>

Commit message: remove collision in URDF

File: romea_camera_description/urdf/camera.xacro (robot description, xacro)
@@ -63,10 +63,10 @@
                 </xacro:if>
             </visual>
-            <collision>
+            <!-- <collision>
                 <origin xyz="${aabb_center[0]} ${aabb_center[1]} ${aabb_center[2]}" rpy="0 0 0" />
                 <geometry>
                 <box size="${aabb_length} ${aabb_width} ${aabb_height}" />
                 </geometry>
-            </collision>
+            </collision> -->
         </link>
         <joint name="${joint_name}" type="fixed">
