Commit message: description: update simulation xacro file
Signed-off-by: jean.laneurit <jean.laneurit@inrae.fr>

File: romea_camera_description/urdf/camera.simulation.xacro (robot description, xacro)
@@ -1,35 +1,35 @@
 <?xml version="1.0"?>
 <robot xmlns:xacro="http://wiki.ros.org/xacro">
-    <xacro:macro name="camera_sensor_simulation"
-      params="prefix mode name link_name configuration ros_namespace">
-        <xacro:property name="image_width"
-          value="${configuration['image_width']}" />
-        <xacro:property name="image_height"
-          value="${configuration['image_height']}" />
-        <xacro:property name="horizontal_fov"
-          value="${configuration['horizontal_fov']}" />
-        <xacro:property name="frame_rate"
-          value="${configuration['frame_rate']}" />
-       <xacro:if value="${'gazebo' in mode}">
-        <gazebo reference="${link_name}">
-          <material>Gazebo/Purple</material>
-          <sensor type="camera" name="${prefix}${name}">
-            <update_rate>${frame_rate}</update_rate>
-            <topic>${ros_namespace}/image_raw</topic>
-            <gz_frame_id>${link_name}</gz_frame_id>  <!-- used only with gazebo 6 or lower -->
-            <ignition_frame_id>${link_name}</ignition_frame_id> <!-- used by gazebo 7 or higher-->
-            <camera>
-              <pose>0 0 0 0 0 0</pose>
-              <horizontal_fov>${horizontal_fov}</horizontal_fov>
-              <image>
-                <width>${image_width} </width>
-                <height>${image_height}</height>
-                <format>R8G8B8</format>
-              </image>
-              <clip>
-                <near>0.01</near>
-                <far>100</far>
-              </clip>
-              <!-- <noise>
+  <xacro:macro name="camera_sensor_simulation"
+    params="prefix mode name link_name configuration ros_namespace">
+    <xacro:property name="image_width"
+      value="${configuration['image_width']}" />
+    <xacro:property name="image_height"
+      value="${configuration['image_height']}" />
+    <xacro:property name="horizontal_fov"
+      value="${configuration['horizontal_fov']}" />
+    <xacro:property name="frame_rate"
+      value="${configuration['frame_rate']}" />
+    <xacro:if value="${'gazebo' in mode}">
+      <gazebo reference="${link_name}">
+        <material>Gazebo/Purple</material>
+        <sensor type="camera" name="${prefix}${name}">
+          <update_rate>${frame_rate}</update_rate>
+          <topic>${ros_namespace}/image_raw</topic>
+          <gz_frame_id>${link_name}</gz_frame_id>  <!-- used only with gazebo 6 or lower -->
+          <ignition_frame_id>${link_name}</ignition_frame_id> <!-- used by gazebo 7 or higher-->
+          <camera>
+            <pose>0 0 0 0 0 0</pose>
+            <horizontal_fov>${horizontal_fov}</horizontal_fov>
+            <image>
+              <width>${image_width} </width>
+              <height>${image_height}</height>
+              <format>R8G8B8</format>
+            </image>
+            <clip>
+              <near>0.01</near>
+              <far>100</far>
+            </clip>
+            <!-- <noise>
                 <type>gaussian</type>
                 <mean>0.0</mean>
@@ -44,25 +44,25 @@
                 <center>0.5 0.5</center>
               </distortion> -->
-            </camera>
-            <xacro:if value="${'classic' in mode}">
-              <plugin name="driver" filename="libgazebo_ros_camera.so">
-                  <ros>
-                    <namespace>${ros_namespace}</namespace>
-                    <remapping>camera/image_raw:=image_raw</remapping>
-                    <remapping>camera/camera_info:=camera_info</remapping>
-                    <remapping>camera/image_raw/compressed:=image_raw/compressed</remapping>
-                    <remapping>camera/image_raw/compressedDepth:=image_raw/compressedDepth</remapping>
-                    <remapping>camera/image_raw/theora:=image_raw/theora</remapping>
-                  </ros>
-                  <camera_name>camera</camera_name>
-                  <hack_baseline>0.07</hack_baseline>
-              </plugin>
-            </xacro:if>
-          </sensor>
-        </gazebo>
-      </xacro:if>
-      <xacro:if value="${'isaac' in mode}">
-        <!-- add description of sensor and ros_bridge for isac sim-->
-      </xacro:if>
-    </xacro:macro>
+          </camera>
+          <xacro:if value="${'classic' in mode}">
+            <plugin name="driver" filename="libgazebo_ros_camera.so">
+              <ros>
+                <namespace>${ros_namespace}</namespace>
+                <remapping>camera/image_raw:=image_raw</remapping>
+                <remapping>camera/camera_info:=camera_info</remapping>
+                <remapping>camera/image_raw/compressed:=image_raw/compressed</remapping>
+                <remapping>camera/image_raw/compressedDepth:=image_raw/compressedDepth</remapping>
+                <remapping>camera/image_raw/theora:=image_raw/theora</remapping>
+              </ros>
+              <camera_name>camera</camera_name>
+              <hack_baseline>0.07</hack_baseline>
+            </plugin>
+          </xacro:if>
+        </sensor>
+      </gazebo>
+    </xacro:if>
+    <xacro:if value="${'isaac' in mode}">
+      <!-- add description of sensor and ros_bridge for isac sim-->
+    </xacro:if>
+  </xacro:macro>
 </robot>

Commit message: add support of new config file
Signed-off-by: jean.laneurit <jean.laneurit@inrae.fr>

File: romea_camera_description/urdf/camera.simulation.xacro (robot description, xacro)
@@ -8,5 +8,5 @@
       value="${configuration['image_height']}" />
     <xacro:property name="horizontal_fov"
-      value="${configuration['horizontal_fov']}" />
+      value="${configuration['horizontal_fov']/180.*pi}" />
     <xacro:property name="frame_rate"
       value="${configuration['frame_rate']}" />
@@ -23,5 +23,5 @@
             <horizontal_fov>${horizontal_fov}</horizontal_fov>
             <image>
-              <width>${image_width} </width>
+              <width>${image_width}</width>
               <height>${image_height}</height>
               <format>R8G8B8</format>

File: romea_camera_description/urdf/camera.xacro (robot description, xacro)
@@ -1,94 +1,99 @@
 <?xml version="1.0"?>
 <robot xmlns:xacro="http://wiki.ros.org/xacro">
-    <xacro:macro name="camera_sensor"
-      params="prefix mode name configuration geometry xyz rpy parent_link mesh_visual ros_namespace">
-        <xacro:property name="M_PI" value="3.1415926535897931" />
-        <xacro:property name="link_name"
-          value="${prefix}${name}_link" />
-        <xacro:property name="joint_name"
-          value="${prefix}${name}_joint" />
-        <xacro:property name="controller_name"
-          value="${prefix}${name}_controller" />
-        <xacro:property name="parent_link_name"
-          value="${prefix}${parent_link}" />
-        <xacro:property name="optical_frame_name"
-          value="${prefix}${name}_optical_frame"/>
-        <xacro:property name="optical_joint_name"
-          value="${prefix}${name}_optical_joint"/>
-        <xacro:property name="mass"
-          value="${geometry['mass']}" />
-        <xacro:property name="aabb"
-          value="${geometry['aabb']}" />
-        <xacro:property name="aabb_length"
-          value="${geometry['aabb']['length']}" />
-        <xacro:property name="aabb_width"
-          value="${geometry['aabb']['width']}" />
-        <xacro:property name="aabb_height"
-          value="${geometry['aabb']['height']}" />
-        <xacro:property name="aabb_center"
-          value="${geometry['aabb']['center']}" />
+  <xacro:macro name="camera_sensor"
+    params="prefix mode name configuration geometry mesh_visual ros_namespace">
+    <xacro:property name="M_PI" value="3.1415926535897931" />
+    <xacro:property name="link_name"
+      value="${prefix}${name}_link" />
+    <xacro:property name="joint_name"
+      value="${prefix}${name}_joint" />
+    <xacro:property name="controller_name"
+      value="${prefix}${name}_controller" />
+    <xacro:property name="parent_link_name"
+      value="${prefix}${configuration['parent_link']}" />
+    <xacro:property name="optical_frame_name"
+      value="${prefix}${name}_optical_frame" />
+    <xacro:property name="optical_joint_name"
+      value="${prefix}${name}_optical_joint" />
+    <xacro:property name="xyz"
+      value="${configuration['xyz']}" />
+    <xacro:property name="rpy"
+      value="${configuration['rpy']}" />
+    <xacro:property name="mass"
+      value="${geometry['mass']}" />
+    <xacro:property name="aabb"
+      value="${geometry['aabb']}" />
+    <xacro:property name="aabb_length"
+      value="${geometry['aabb']['length']}" />
+    <xacro:property name="aabb_width"
+      value="${geometry['aabb']['width']}" />
+    <xacro:property name="aabb_height"
+      value="${geometry['aabb']['height']}" />
+    <xacro:property name="aabb_center"
+      value="${geometry['aabb']['center']}" />
+    <xacro:if value="${mesh_visual == True and 'mesh' in geometry}">
+      <xacro:property name="mesh_xyz"
+        value="${geometry['mesh']['xyz']}" />
+      <xacro:property name="mesh_rpy"
+        value="${geometry['mesh']['rpy']}" />
+      <xacro:property name="mesh_scale"
+        value="${geometry['mesh']['scale']}" />
+      <xacro:property name="mesh_filename"
+        value="${geometry['mesh']['filename']}" />
+    </xacro:if>
+    <link name="${link_name}">
+      <inertial>
+        <mass value="${mass}" />
+        <origin xyz="${aabb_center[0]} ${aabb_center[1]} ${aabb_center[2]}" />
+        <inertia ixx="${0.0833333 * mass * (aabb_width*aabb_width + aabb_height*aabb_height)}"
+          ixy="0.0" ixz="0.0"
+          iyy="${0.0833333 * mass * (aabb_height*aabb_height + aabb_length*aabb_length)}" iyz="0.0"
+          izz="${0.0833333 * mass * (aabb_length*aabb_length + aabb_width*aabb_width)}" />
+      </inertial>
+      <visual>
         <xacro:if value="${mesh_visual == True and 'mesh' in geometry}">
-          <xacro:property name="mesh_xyz"
-            value="${geometry['mesh']['xyz']}" />
-          <xacro:property name="mesh_rpy"
-            value="${geometry['mesh']['rpy']}" />
-          <xacro:property name="mesh_scale"
-            value="${geometry['mesh']['scale']}" />
-          <xacro:property name="mesh_filename"
-            value="${geometry['mesh']['filename']}" />
+          <origin xyz="${mesh_xyz[0]} ${mesh_xyz[1]} ${mesh_xyz[2]}"
+            rpy="${mesh_rpy[0]/180.*pi} ${mesh_rpy[1]/180.*pi} ${mesh_rpy[2]/180.*pi}" />
+          <geometry>
+            <mesh filename="${mesh_filename}"
+              scale="${mesh_scale[0]} ${mesh_scale[1]} ${mesh_scale[2]}" />
+          </geometry>
         </xacro:if>
-        <link name="${link_name}">
-            <inertial>
-                <mass value="${mass}" />
-                <origin xyz="${aabb_center[0]} ${aabb_center[1]} ${aabb_center[2]}" />
-                <inertia ixx="${0.0833333 * mass * (aabb_width*aabb_width + aabb_height*aabb_height)}"
-                ixy="0.0" ixz="0.0"
-                iyy="${0.0833333 * mass * (aabb_height*aabb_height + aabb_length*aabb_length)}" iyz="0.0"
-                izz="${0.0833333 * mass * (aabb_length*aabb_length + aabb_width*aabb_width)}" />
-            </inertial>
-            <visual>
-                <xacro:if value="${mesh_visual == True and 'mesh' in geometry}">
-                    <origin xyz="${mesh_xyz[0]} ${mesh_xyz[1]} ${mesh_xyz[2]}"
-                        rpy="${mesh_rpy[0]} ${mesh_rpy[1]} ${mesh_rpy[2]}" />
-                    <geometry>
-                        <mesh filename="${mesh_filename}"
-                        scale="${mesh_scale[0]} ${mesh_scale[1]} ${mesh_scale[2]}" />
-                    </geometry>
-                </xacro:if>
-                <xacro:if value="${mesh_visual == False or 'mesh' not in geometry}">
-                    <origin xyz="${aabb_center[0]} ${aabb_center[1]} ${aabb_center[2]}" rpy="0 0 0" />
-                    <geometry>
-                        <box size="${aabb_length} ${aabb_width} ${aabb_height}" />
-                    </geometry>
-                </xacro:if>
-            </visual>
-            <!-- <collision>
-                <origin xyz="${aabb_center[0]} ${aabb_center[1]} ${aabb_center[2]}" rpy="0 0 0" />
-                <geometry>
-                <box size="${aabb_length} ${aabb_width} ${aabb_height}" />
-                </geometry>
-            </collision> -->
-        </link>
-        <joint name="${joint_name}" type="fixed">
-            <parent link="${parent_link_name}"/>
-            <child link="${link_name}"/>
-            <origin xyz="${xyz}" rpy="${rpy}" />
-        </joint>
-        <link name="${optical_frame_name}"/>
-        <joint name="${optical_joint_name}" type="fixed">
-            <origin xyz="0 0 0" rpy="-${M_PI/2} 0.0 -${M_PI/2}"/>
-            <parent link="${link_name}"/>
-            <child link="${optical_frame_name}"/>
-        </joint>
-        <xacro:if value="${'simulation' in mode}">
-          <xacro:include filename="$(find romea_camera_description)/urdf/camera.simulation.xacro" />
-            <xacro:camera_sensor_simulation
-              prefix="${prefix}"
-              mode="${mode}"
-              name="${name}"
-              link_name="${link_name}"
-              configuration="${configuration}"
-              ros_namespace="${ros_namespace}"/>
+        <xacro:if value="${mesh_visual == False or 'mesh' not in geometry}">
+          <origin xyz="${aabb_center[0]} ${aabb_center[1]} ${aabb_center[2]}" rpy="0 0 0" />
+          <geometry>
+            <box size="${aabb_length} ${aabb_width} ${aabb_height}" />
+          </geometry>
         </xacro:if>
-    </xacro:macro>
+      </visual>
+      <!-- <collision>
+        <origin xyz="${aabb_center[0]} ${aabb_center[1]} ${aabb_center[2]}" rpy="0 0 0" />
+        <geometry>
+          <box size="${aabb_length} ${aabb_width} ${aabb_height}" />
+        </geometry>
+      </collision> -->
+    </link>
+    <joint name="${joint_name}" type="fixed">
+      <parent link="${parent_link_name}" />
+      <child link="${link_name}" />
+      <origin xyz="${xyz[0]} ${xyz[1]} ${xyz[2]}"
+        rpy="${rpy[0]/180.*pi} ${rpy[1]/180.*pi} ${rpy[2]/180.*pi}" />
+    </joint>
+    <link name="${optical_frame_name}" />
+    <joint name="${optical_joint_name}" type="fixed">
+      <origin xyz="0 0 0" rpy="-${M_PI/2} 0.0 -${M_PI/2}" />
+      <parent link="${link_name}" />
+      <child link="${optical_frame_name}" />
+    </joint>
+    <xacro:if value="${'simulation' in mode}">
+      <xacro:include filename="$(find romea_camera_description)/urdf/camera.simulation.xacro" />
+      <xacro:camera_sensor_simulation
+        prefix="${prefix}"
+        mode="${mode}"
+        name="${name}"
+        link_name="${link_name}"
+        configuration="${configuration}"
+        ros_namespace="${ros_namespace}" />
+    </xacro:if>
+  </xacro:macro>
 </robot>
