Commit message: merge romea_camera + romea_stereo_camera + romea_rgbd_camera
Signed-off-by: jean.laneurit <jean.laneurit@inrae.fr>

File: romea_camera_description/urdf/monocular_camera.simulation.xacro (robot description, xacro)
@@ -1,5 +1,5 @@
 <?xml version="1.0"?>
 <robot xmlns:xacro="http://wiki.ros.org/xacro">
-  <xacro:macro name="camera_sensor_simulation"
+  <xacro:macro name="monocular_camera_sensor_simulation"
     params="prefix mode name link_name configuration ros_namespace">
     <xacro:property name="image_width"

File: romea_camera_description/urdf/monocular_camera.xacro (robot description, xacro)
@@ -3,5 +3,4 @@
   <xacro:macro name="camera_sensor"
     params="prefix mode name configuration geometry mesh_visual ros_namespace">
-    <xacro:property name="M_PI" value="3.1415926535897931" />
     <xacro:property name="link_name"
       value="${prefix}${name}_link" />
@@ -82,11 +81,12 @@
     <link name="${optical_frame_name}" />
     <joint name="${optical_joint_name}" type="fixed">
-      <origin xyz="0 0 0" rpy="-${M_PI/2} 0.0 -${M_PI/2}" />
+      <origin xyz="0 0 0" rpy="-${pi/2} 0.0 -${pi/2}" />
       <parent link="${link_name}" />
       <child link="${optical_frame_name}" />
     </joint>
     <xacro:if value="${'simulation' in mode}">
-      <xacro:include filename="$(find romea_camera_description)/urdf/camera.simulation.xacro" />
-      <xacro:camera_sensor_simulation
+      <xacro:include
+        filename="$(find romea_camera_description)/urdf/monocular_camera.simulation.xacro" />
+      <xacro:monocular_camera_sensor_simulation
         prefix="${prefix}"
         mode="${mode}"
