Commit message: add simulation test + gz_bridge
Signed-off-by: Jean Laneurit <jean.laneurit@inrae.fr>

File: romea_camera_description/urdf/monocular_camera.xacro (robot description, xacro)
@@ -2,5 +2,5 @@
 <robot xmlns:xacro="http://wiki.ros.org/xacro">
   <xacro:macro name="camera_sensor"
-    params="prefix mode name configuration geometry mesh_visual ros_namespace">
+    params="prefix mode name configuration geometry mesh_visual ros_namespace standalone">
     <xacro:property name="link_name"
       value="${prefix}${name}_link" />
@@ -73,10 +73,12 @@
       </collision> -->
     </link>
-    <joint name="${joint_name}" type="fixed">
-      <parent link="${parent_link_name}" />
-      <child link="${link_name}" />
-      <origin xyz="${xyz[0]} ${xyz[1]} ${xyz[2]}"
-        rpy="${rpy[0]/180.*pi} ${rpy[1]/180.*pi} ${rpy[2]/180.*pi}" />
-    </joint>
+    <xacro:if value="${standalone == False}">
+      <joint name="${joint_name}" type="fixed">
+        <parent link="${parent_link_name}" />
+        <child link="${link_name}" />
+        <origin xyz="${xyz[0]} ${xyz[1]} ${xyz[2]}"
+          rpy="${rpy[0]/180.*pi} ${rpy[1]/180.*pi} ${rpy[2]/180.*pi}" />
+      </joint>
+    </xacro:if>
     <link name="${optical_frame_name}" />
     <joint name="${optical_joint_name}" type="fixed">

File: romea_camera_description/urdf/stereo_camera.simulation.xacro (robot description, xacro)
@@ -2,5 +2,5 @@
 <robot xmlns:xacro="http://wiki.ros.org/xacro">
   <xacro:macro name="camera_stereo_sensor_simulation"
-    params="prefix mode name link_name configuration ros_namespace">
+    params="prefix mode name baseline link_name left_camera_link_name right_camera_link_name configuration ros_namespace">
     <xacro:property name="image_width"
       value="${configuration['image_width']}" />
@@ -11,4 +11,73 @@
     <xacro:property name="frame_rate"
       value="${configuration['frame_rate']}" />
+    <xacro:if value="${'gazebo_classic' not in  mode}">
+      <gazebo reference="${link_name}">
+        <material>Gazebo/DarkYellow </material>
+        <sensor type="camera" name="${prefix}${name}_left_camera">
+          <update_rate>${frame_rate}</update_rate>
+          <topic>${ros_namespace}/left/image_raw</topic>
+          <gz_frame_id>${left_camera_link_name}</gz_frame_id>  <!-- used only with gazebo 6 or lower -->
+          <ignition_frame_id>${left_camera_link_name}</ignition_frame_id> <!-- used by gazebo 7 or higher-->
+          <camera>
+            <pose>0 -${baseline/2} 0 0 0 0</pose>
+            <horizontal_fov>${horizontal_fov}</horizontal_fov>
+            <image>
+              <width>${image_width}</width>
+              <height>${image_height}</height>
+              <format>R8G8B8</format>
+            </image>
+            <clip>
+              <near>0.01</near>
+              <far>100</far>
+            </clip>
+            <!-- <noise>
+                <type>gaussian</type>
+                <mean>0.0</mean>
+                <stddev>0.007</stddev>
+              </noise>
+              <distortion>
+                <k1>0.0</k1>
+                <k2>0.0</k2>
+                <k3>0.0</k3>
+                <p1>0.0</p1>
+                <p2>0.0</p2>
+                <center>0.5 0.5</center>
+              </distortion> -->
+          </camera>
+        </sensor>
+        <sensor type="camera" name="${prefix}${name}_right_camera">
+          <update_rate>${frame_rate}</update_rate>
+          <topic>${ros_namespace}/right/image_raw</topic>
+          <gz_frame_id>${right_camera_link_name}</gz_frame_id>  <!-- used only with gazebo 6 or lower -->
+          <ignition_frame_id>${right_camera_link_name}</ignition_frame_id> <!-- used by gazebo 7 or higher-->
+          <camera>
+            <pose>0 ${baseline/2} 0 0 0 0</pose>
+            <horizontal_fov>${horizontal_fov}</horizontal_fov>
+            <image>
+              <width>${image_width}</width>
+              <height>${image_height}</height>
+              <format>R8G8B8</format>
+            </image>
+            <clip>
+              <near>0.01</near>
+              <far>100</far>
+            </clip>
+            <!-- <noise>
+                <type>gaussian</type>
+                <mean>0.0</mean>
+                <stddev>0.007</stddev>
+              </noise>
+              <distortion>
+                <k1>0.0</k1>
+                <k2>0.0</k2>
+                <k3>0.0</k3>
+                <p1>0.0</p1>
+                <p2>0.0</p2>
+                <center>0.5 0.5</center>
+              </distortion> -->
+          </camera>
+        </sensor>
+      </gazebo>
+    </xacro:if>
     <xacro:if value="${'gazebo_classic' in  mode}">
       <gazebo reference="${link_name}">

File: romea_camera_description/urdf/stereo_camera.xacro (robot description, xacro)
@@ -2,5 +2,5 @@
 <robot xmlns:xacro="http://wiki.ros.org/xacro">
   <xacro:macro name="camera_sensor"
-    params="prefix mode name configuration geometry mesh_visual ros_namespace">
+    params="prefix mode name configuration geometry mesh_visual ros_namespace standalone">
     <xacro:property name="link_name"
       value="${prefix}${name}_link" />
@@ -54,10 +54,12 @@
     </xacro:if>
     <!-- Camera Center -->
-    <joint name="${joint_name}" type="fixed">
-      <parent link="${parent_link_name}" />
-      <child link="${link_name}" />
-      <origin xyz="${xyz[0]} ${xyz[1]} ${xyz[2]}"
-        rpy="${rpy[0]/180.*pi} ${rpy[1]/180.*pi} ${rpy[2]/180.*pi}" />
-    </joint>
+    <xacro:if value="${standalone == False}">
+      <joint name="${joint_name}" type="fixed">
+        <parent link="${parent_link_name}" />
+        <child link="${link_name}" />
+        <origin xyz="${xyz[0]} ${xyz[1]} ${xyz[2]}"
+          rpy="${rpy[0]/180.*pi} ${rpy[1]/180.*pi} ${rpy[2]/180.*pi}" />
+      </joint>
+    </xacro:if>
     <link name="${link_name}">
       <inertial>
@@ -125,5 +127,8 @@
         mode="${mode}"
         name="${name}"
+        baseline="${baseline}"
         link_name="${link_name}"
+        left_camera_link_name="${left_camera_link_name}"
+        right_camera_link_name="${right_camera_link_name}"
         configuration="${configuration}"
         ros_namespace="${ros_namespace}" />
